File: Memory/24LC256.brd (EAGLE design)
At the start: 16.8 x 13.3 mm, 4 parts

Commit message: new boards
Parts:
- removed 100NF: 100nF, SparkFun-Capacitors:0603-CAP
- removed J1, J2: (no value), SparkFun-Connectors:1X04
- removed U$1: TSL230RDSMD, awqua_eagle_library:TSL230RD
- added C_100N: 100n, SparkFun:0603-CAP
- added FRAME1: FRAME-LETTER, SparkFun-Aesthetics:CREATIVE_COMMONS
- added JP1: (no value), SparkFun-Connectors:1X04
- added R1,R2=10K, R1_10K: (no value), SparkFun-Passives:0603-RES
- added U2: EEPROM-I2CSMD, SparkFun-DigitalIC:SO08
Connections:
- removed net N$1: J2.4, U$1.S0
- removed net N$2: J2.3, U$1.S1
- removed net N$3: J2.2, U$1.OE
- removed net N$5: J1.1, U$1.S3
- removed net N$6: J1.2, U$1.S2
- removed net N$7: J1.3, U$1.OUT
- removed net N$8: 100NF.1, J1.4, U$1.VDD
- new net SCL: JP1.3, R1_10K.1, U2.6
- new net SDA: JP1.4, R1,R2=10K.1, U2.5
- new net VCC: C_100N.1, JP1.1, R1,R2=10K.2, R1_10K.2, U2.8
- net GND: now also C_100N.2, JP1.2, U2.1, U2.2, U2.3, U2.4, U2.7; no longer 100NF.2, J2.1, U$1.GND
Routing:
- net VCC: track 0.00 -> 23.1 mm, vias 0 -> 2
- net SDA: track 0.00 -> 10.9 mm
- net GND: track 7.22 -> 15.5 mm, vias 0 -> 1
- net N$8: track 7.54 -> 0.00 mm
- net SCL: track 0.00 -> 6.72 mm
- net N$7: track 3.62 -> 0.00 mm
- net N$3: track 3.34 -> 0.00 mm
- net N$5: track 3.22 -> 0.00 mm
- net N$6: track 3.15 -> 0.00 mm
- net N$1: track 2.91 -> 0.00 mm
- net N$2: track 2.85 -> 0.00 mm
Other:
- board size 16.8 x 13.3 mm -> 16.5 x 12.2 mm
- board text added: "*"
- board text added: "Chris Kelley / AWQUA"
- board text added: "SCL"
- board text added: "SDA"
- board text added: "VCC"
- board text removed: "OE"
- board text removed: "OUT"
- board text removed: "S0"
- board text removed: "S1"
- board text removed: "S2"
- board text removed: "S3"
- board text removed: "TSL230RD V1.0, 2016/02/25, A.B."
- board text removed: "VDD"
