File: RTC/DS3231.brd (EAGLE design)
At the start: 16.8 x 13.3 mm, 4 parts

Commit message: new boards
Parts:
- removed 100NF: 100nF, SparkFun-Capacitors:0603-CAP
- removed J1, J2: (no value), SparkFun-Connectors:1X04
- removed U$1: TSL230RDSMD, awqua_eagle_library:TSL230RD
- added C_100N: 100n, SparkFun:0603-CAP
- added DS3231: (no value), open_source_turbidimeter:DS3231M
- added FRAME1: FRAME-LETTER, SparkFun-Aesthetics:CREATIVE_COMMONS
- added JP1: (no value), SparkFun-Connectors:1X06
- added PAD1, PAD2, PAD3, PAD4: WIREPADSMD5-2,5, wirepad:5-2,5
- added R1_10K, R2_10K: (no value), SparkFun-Passives:0603-RES
Connections:
- removed net N$1: J2.4, U$1.S0
- removed net N$2: J2.3, U$1.S1
- removed net N$3: J2.2, U$1.OE
- removed net N$5: J1.1, U$1.S3
- removed net N$6: J1.2, U$1.S2
- removed net N$7: J1.3, U$1.OUT
- removed net N$8: 100NF.1, J1.4, U$1.VDD
- new net SCL: DS3231.8, JP1.5, R1_10K.1
- new net SDA: DS3231.7, JP1.6, R2_10K.1
- new net SQW: DS3231.3, JP1.2
- new net VBAT: C_100N.2, DS3231.6, PAD1.1, PAD2.1
- new net VCC: DS3231.2, JP1.4, R1_10K.2, R2_10K.2
- net GND: now also C_100N.1, DS3231.5, JP1.1, JP1.3, PAD3.1, PAD4.1; no longer 100NF.2, J2.1, U$1.GND
Routing:
- net VBAT: track 0.00 -> 52.3 mm, vias 0 -> 1
- net VCC: track 0.00 -> 16.6 mm
- net SDA: track 0.00 -> 13.9 mm
- net SQW: track 0.00 -> 13.9 mm
- net SCL: track 0.00 -> 9.37 mm
- net N$8: track 7.54 -> 0.00 mm
- net N$7: track 3.62 -> 0.00 mm
- net N$3: track 3.34 -> 0.00 mm
- net N$5: track 3.22 -> 0.00 mm
- net N$6: track 3.15 -> 0.00 mm
- net N$1: track 2.91 -> 0.00 mm
- net N$2: track 2.85 -> 0.00 mm
- net GND: track 7.22 -> 6.56 mm, vias 0 -> 1
- added copper zone on layer 1, net GND
- removed copper zone on layer 16, net GND
Other:
- board size 16.8 x 13.3 mm -> 25.4 x 19.3 mm
- board text added: "*"
- board text added: "Chris Kelley / AWQUA"
- board text added: "SCL"
- board text added: "SDA"
- board text added: "SQW"
- board text added: "VCC"
- board text removed: "OE"
- board text removed: "OUT"
- board text removed: "S0"
- board text removed: "S1"
- board text removed: "S2"
- board text removed: "S3"
- board text removed: "TSL230RD V1.0, 2016/02/25, A.B."
- board text removed: "VDD"
